Commit message: realised physics engine won't work

File: robot.urdf (robot description, URDF)
Before this commit: robot None, 7 links, 6 joints
Links:
- link 5: geometry collision box size=0.15 0.05 0.15; visual box size=0.15 0.05 0.15
- link 6: geometry collision box size=0.15 0.05 0.125; visual box size=0.15 0.05 0.125
Joints:
- removed joint gripper
- joint : origin xyz=0 0.075 0 rpy=1.5707963267948966 0 0 -> xyz=0 -0.075 0.15 rpy=1.5707963057214724 0 0
- joint elbow: limit lower=-2.5132741228718345 upper=2.5132741228718345 effort=0 velocity=10 -> lower=-2.5132741228718345 upper=2.5132741228718345 effort=100 velocity=10; origin xyz=0 -0.075 0.3 rpy=1.5707963267948966 0 0 -> xyz=0 0.075 0.65 rpy=-1.5707963057214724 0 0
- joint lift: axis 0 0 -1 -> 0 1 0; limit lower=0 upper=1500 effort=0 velocity=10 -> lower=0 upper=1.5 effort=100 velocity=10; origin xyz=0 -0.075 1 rpy=1.5707963267948966 0 0 -> xyz=0 0.075 1.925 rpy=-1.5707963057214724 0 0
- joint swing: limit lower=-3.141592653589793 upper=3.141592653589793 effort=0 velocity=10 -> lower=-3.141592653589793 upper=3.141592653589793 effort=100 velocity=10
- joint wrist: limit lower=-3.141592653589793 upper=3.141592653589793 effort=0 velocity=10 -> lower=-3.141592653589793 upper=3.141592653589793 effort=100 velocity=10; origin xyz=0 -0.075 0.3 rpy=1.5707963267948966 0 0 -> xyz=0 -0.6 0.15000000000000005 rpy=-1.1102230246251565e-16 0 0

Commit message: tried using k ik solver

File: robot.urdf (robot description, URDF)
Before this commit: robot None, 7 links, 5 joints
Joints:
- added joint gripper: type prismatic, parent 5, child 6, origin xyz=0 0.025 0.125 rpy=-1.5707963057214724 0 0, axis 0 1 0, limit lower=0 upper=0.1 effort=100 velocity=0.1
- joint elbow: limit lower=-2.5132741228718345 upper=2.5132741228718345 effort=100 velocity=10 -> lower=-8594.366926962348 upper=8594.366926962348 effort=100 velocity=1145.9155902616465
- joint lift: limit lower=0 upper=1.5 effort=100 velocity=10 -> lower=0 upper=1.5 effort=100 velocity=0.1
- joint swing: limit lower=-3.141592653589793 upper=3.141592653589793 effort=100 velocity=10 -> lower=-10313.240312354817 upper=10313.240312354817 effort=100 velocity=1145.9155902616465
- joint wrist: limit lower=-3.141592653589793 upper=3.141592653589793 effort=100 velocity=10 -> lower=-10313.240312354817 upper=10313.240312354817 effort=100 velocity=1145.9155902616465
